File: hardware/schematic/BedMCU.kicad_pcb (KiCad board)
At the start: 4 copper layers, 80 x 80 mm, 170 parts, among them J1 2.54-2P, J10 5.0-2P, J11 2.54-2P, J12 2.54-2P, J13 2.54-2P, J14 2.54-2P, J15 2.54-2X6P, J16 918-518K2023S50000, J17 2.54-2P, J18 918-518K2023S50000, J19 47053-1000, J2 2.54-2P, J3 XT30PW(2+2)-M, J4 PZ254V-11-02P, J5 2.54-4P, J6 2.54-4P, J7 2.54-4P, J8 2.54-4P, J9 5.0-2P, Q1 HYG017N04LS1C2, Q2 HYG017N04LS1C2, Q3 PNMT30V6, SW1 TSA016A2518A, SW2 TSA016A2518A, SW3 TSA016A2518A, SW4 TSA016A2518A, U1 TPS5430DDAR, U10 TJA1051TK/3/1J, U11 RP2040, U12 74HCT365D,653, U2 AMS1117-3.3, U3 INA350ABSIDDFR, U4 W25Q16JVUXIQ, U5 TPS76925DBVR, U6 TLV333, U7 RP2040, U8 W25Q16JVUXIQ, U9 ADXL345BCCZ, X1 X322512MSB4SI, X2 X322512MSB4SI

Commit message: fix: correct symbol for op amp
Connections:
- U6 pad 2: (no net) -> GND
- U6 pad 4: GND -> Net-(U6-IN-)

Commit message: feat: upload rev 3.1 schematic
Parts:
- C1, C44: value 100n -> 100nF
- J1, J11, J12, J13, J14, J17, J2: value 2.54-2P -> 2.54-2P ZZDK
- J10, J9: value 5.0-2P -> DB301V-5.0-2P
- J15: value 2.54-2X6P -> KH-2.54PH180-2X6P-L8.9
- J5, J6, J7, J8: value 2.54-4P -> XY308-2.54-4P
- moved R16 4.03 mm to (159.6, 68.3), turned to -90 degrees
- moved R12 3.72 mm to (164.6, 67.7)
- moved TP23 1.75 mm to (160.4, 70.5)
- moved R13 1.60 mm to (165.6, 69.0)
- moved C14 1.60 mm to (161.5, 65.4)
- moved U6 1.60 mm to (162.0, 67.8)
- moved R15 1.50 mm to (164.1, 69.5)
- moved TP24 1.39 mm to (168.4, 69.0)
- moved TP21 0.20 mm to (149.3, 67.5)
- moved TP26 0.10 mm to (168.8, 75.4)
Routing:
- net Net-(U6-IN-): track 1.13 -> 5.82 mm
- net /Sensors/WGT_OUT: track 8.17 -> 6.62 mm
- net /Sensors/2V5_REF: track 66.7 -> 67.8 mm
- net /Sensors/WGT_PRE: track 4.34 -> 4.85 mm
- net GND: vias 162 -> 165
Other:
- board text added: "Bed MCU Rev 3.1 by eliteSCHW31N"
- board text added: "TP1 : ${3630b6a0-46fc-4978-9b5b-b87ac7104fcd:NET_NAME(1)} TP2 : ${e9d94a36-d374-41d5-8e0e-96e27e30d585:NET_NAME(1)} TP3 : ${5e741447-af0f-45b6-b0a0-e2b92af4a012:NET_NAME(1)} TP4 : ${2c3026d7-e455-46ae-9ae1-6638e1bac7d3:NET_NAME(1)} TP5 : ${a2e152f2-b34a-4058-bbdb-c6c542840e1b:SHORT_NET_NAME(1)} TP6 : ${9941992e-487d-49d0-b769-cac432bf3cf1:SHORT_NET_NAME(1)} TP7 : ${4c75d921-17c7-4c81-8b4d-10ade82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"
- board text added: "TP15 : ${e37f7efe-5b44-4324-b579-213a97d4b845:NET_NAME(1)} TP16 : ${a14c5b00-80f1-4668-8c77-818c92d709a1:NET_NAME(1)} TP17 : ${2cd55360-432d-4f7a-8025-e2ae73fd2658:NET_NAME(1)} TP18 : ${5608abae-59fd-4909-bfd0-e8e968239170:NET_NAME(1)} TP19 : ${2aaa11d9-89d6-4b47-8292-f2800353f813:NET_NAME(1)} TP20 : ${2d10b2b5-a566-4b9b-97bf-e2ec93a9a855:NET_NAME(1)} TP21 : ${c062707c-b811-438c-a85e-06958382acb4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"
- board text removed: "Bed MCU Rev 3.0 by eliteSCHW31N"
