File: hardware/schematic/power.kicad_sch (KiCad schematic)
At the start: 31 parts, among them J1 2.54-2P, J2 2.54-2P, J3 XT30PW(2+2)-M, U1 TPS5430DDAR, U2 AMS1117-3.3

Commit message: feat: upload rev 3.1 schematic
Parts:
- C1: value 100n -> 100nF
- J1, J2: value 2.54-2P -> 2.54-2P ZZDK; LCSC Part (none) -> C18185649
- TP1, TP2, TP3, TP4: now in the parts list
Connections:
- no-connect marks 2 -> 0
Other:
- moved on the sheet: C1, C2, C3, C7, C8, D4, J1, J2, L1, R1, R4, R6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
