File: hardware/schematic/usb.kicad_sch (KiCad schematic)
At the start: 9 parts, among them J16 918-518K2023S50000, J17 2.54-2P, J18 918-518K2023S50000

Commit message: feat: upload rev 3.1 schematic
Parts:
- J17: value 2.54-2P -> 2.54-2P ZZDK; LCSC Part (none) -> C18185649
- TP5: now in the parts list
Other:
- moved on the sheet: D8, J17, J18, R33, R34, R35, R36
